Commit message: feat: Project submsion

File: workspace/catkin_ws/src/my_robot/urdf/my_robot.xacro (robot description, xacro)
@@ -32,4 +32,9 @@
     <dynamics damping="1.0" friction="1.0"/>
   </joint>
+  <joint name="camera_optical_joint" type="fixed">
+    <origin xyz="0 0 0" rpy="-1.5707 0 -1.5707"/>
+    <parent link="camera"/>
+    <child link="camera_link_optical"/>
+  </joint>
   <joint type="fixed" name="hokuyo_joint">
     <origin xyz="0.15 0 0.1" rpy="0 0 0"/>
@@ -63,4 +68,6 @@
     </visual>
   </link>
+  <link name="camera_link_optical">
+  </link>
   <link name='camera'>
     <inertial>
